Commit message: Added end effector groups to SRDF xacro

File: baxter/baxter_moveit_config/config/baxter_base.srdf.xacro (robot description, xacro)
@@ -24,13 +24,12 @@
     </group>
     <group name="left_hand">
-        <link name="left_hand" />
-        <link name="left_gripper_base" />
-        <link name="left_gripper" />
+        <chain base_link="left_hand" tip_link="$(arg left_tip_name)" />
     </group>
     <group name="right_hand">
-        <link name="right_hand" />
-        <link name="right_gripper_base" />
-        <link name="right_gripper" />
-    </group>
+        <chain base_link="right_hand" tip_link="$(arg right_tip_name)" />
+    </group>
+    <!--END EFFECTOR: Purpose: Represent information about an end effector.-->
+    <end_effector name="left_hand_eef" parent_link="$(arg left_tip_name)" group="left_hand" parent_group="left_arm" />
+    <end_effector name="right_hand_eef" parent_link="$(arg right_tip_name)" group="right_hand" parent_group="right_arm" />
     <!--GROUP STATES: Purpose: Define a named state for a particular group, in terms of joint values. This is useful to define states like 'folded arms'-->
     <group_state name="left_neutral" group="left_arm">
@@ -53,6 +52,4 @@
     </group_state>
     <!--END EFFECTOR: Purpose: Represent information about an end effector.-->
-    <end_effector name="left_hand_eef" parent_link="left_gripper" group="left_hand" parent_group="left_arm" />
-    <end_effector name="right_hand_eef" parent_link="right_gripper" group="right_hand" parent_group="right_arm" />
      <!--VIRTUAL JOINT: Purpose: this element defines a virtual joint between a robot link and an external frame of reference (considered fixed with respect to the robot)-->
     <virtual_joint name="world_joint" type="floating" parent_frame="world" child_link="torso" />

File: baxter/baxter_moveit_config/config/rethink_electric_gripper.srdf.xacro (robot description, xacro)
@@ -73,5 +73,8 @@
     <disable_collisions link1="${side}_gripper_r_finger_tip" link2="${side}_upper_forearm_visual" reason="Never" />
     <disable_collisions link1="${side}_gripper_r_finger_tip" link2="${side}_wrist" reason="Never" />
-    <disable_collisions link1="${side}_gripper_l_finger_tip" link2="${side}_gripper_r_finger_tip" reason="Adjacent" />
+    <disable_collisions link1="${side}_gripper_l_finger_tip" link2="${side}_gripper_r_finger_tip" reason="Never" />
+    <disable_collisions link1="${side}_gripper_l_finger" link2="${side}_gripper_l_finger_tip" reason="Never" />
+    <disable_collisions link1="${side}_gripper_r_finger" link2="${side}_gripper_r_finger_tip" reason="Never" />
+    <disable_collisions link1="${side}_gripper_base" link2="${side}_gripper_electric_base" reason="Never" />
     </xacro:macro>
 </robot>
