Commit message: Fixed electric gripper configurations for SRDFs
- Now a default end effector sdf takes care of the default <side>_gripper
  collisions
- Electric Gripper specific collisions use the correct finger link names
- Set the default tip name to be <side>_gripper
- Fixed a move_group arg value in demo_baxter
- Removed nefarious planning_context.launch call from move_group.launch
  which would overwrite all args from a previous move_group.launch call

File: baxter/baxter_moveit_config/config/baxter.srdf.xacro (robot description, xacro)
@@ -5,4 +5,7 @@
   <xacro:include filename="$(find baxter_moveit_config)/config/baxter_base.srdf.xacro" />
   <xacro:baxter_base left_tip_name="$(arg left_tip_name)" right_tip_name="$(arg right_tip_name)"/>
+  <!--Left End Effector Collisions-->
+  <xacro:include filename="$(find baxter_moveit_config)/config/default_gripper.srdf.xacro" />
+  <xacro:default_gripper side="left"/>
   <xacro:arg name="left_electric_gripper" default="false"/>
   <xacro:if value="$(arg left_electric_gripper)">
@@ -10,4 +13,7 @@
     <xacro:rethink_electric_gripper side="left"/>
   </xacro:if>
+  <!--Right End Effector Collisions-->
+  <xacro:include filename="$(find baxter_moveit_config)/config/default_gripper.srdf.xacro" />
+  <xacro:default_gripper side="right"/>
   <xacro:arg name="right_electric_gripper" default="false"/>
   <xacro:if value="$(arg right_electric_gripper)">

File: baxter/baxter_moveit_config/config/baxter_base.srdf.xacro (robot description, xacro)
@@ -76,5 +76,4 @@
     <disable_collisions link1="collision_head_link_2" link2="sonar_ring" reason="Never" />
     <disable_collisions link1="collision_head_link_2" link2="torso" reason="Adjacent" />
-    <disable_collisions link1="head" link2="left_gripper" reason="Never" />
     <disable_collisions link1="head" link2="left_hand_camera" reason="Never" />
     <disable_collisions link1="head" link2="left_hand_range" reason="Never" />
@@ -84,5 +83,4 @@
     <disable_collisions link1="head" link2="left_upper_shoulder" reason="Never" />
     <disable_collisions link1="head" link2="pedestal" reason="Never" />
-    <disable_collisions link1="head" link2="right_gripper" reason="Never" />
     <disable_collisions link1="head" link2="right_hand_camera" reason="Never" />
     <disable_collisions link1="head" link2="right_hand_range" reason="Never" />
@@ -94,20 +92,4 @@
     <disable_collisions link1="head" link2="sonar_ring" reason="Never" />
     <disable_collisions link1="head" link2="torso" reason="Adjacent" />
-    <disable_collisions link1="left_gripper" link2="left_hand" reason="Adjacent" />
-    <disable_collisions link1="left_gripper" link2="left_hand_camera" reason="Never" />
-    <disable_collisions link1="left_gripper" link2="left_hand_range" reason="Never" />
-    <disable_collisions link1="left_gripper" link2="left_lower_elbow" reason="Never" />
-    <disable_collisions link1="left_gripper" link2="left_lower_forearm" reason="Never" />
-    <disable_collisions link1="left_gripper" link2="left_upper_elbow_visual" reason="Never" />
-    <disable_collisions link1="left_gripper" link2="left_upper_forearm" reason="Never" />
-    <disable_collisions link1="left_gripper" link2="left_upper_forearm_visual" reason="Never" />
-    <disable_collisions link1="left_gripper" link2="left_wrist" reason="Never" />
-    <disable_collisions link1="left_gripper" link2="right_hand_camera" reason="Never" />
-    <disable_collisions link1="left_gripper" link2="right_hand_range" reason="Never" />
-    <disable_collisions link1="left_gripper" link2="screen" reason="Never" />
-    <disable_collisions link1="left_gripper" link2="sonar_ring" reason="Never" />
-    <disable_collisions link1="left_gripper" link2="pedestal" reason="Never" />
-    <disable_collisions link1="left_gripper_base" link2="left_hand_accelerometer" reason="Never" />
-    <disable_collisions link1="left_hand" link2="left_gripper_base" reason="Adjacent" />
     <disable_collisions link1="left_hand" link2="left_hand_camera" reason="Adjacent" />
     <disable_collisions link1="left_hand" link2="left_hand_range" reason="Adjacent" />
@@ -138,5 +120,4 @@
     <disable_collisions link1="left_hand_range" link2="left_upper_forearm" reason="Never" />
     <disable_collisions link1="left_wrist" link2="left_hand_accelerometer" reason="Never" />
-    <disable_collisions link1="left_wrist" link2="left_gripper_base" reason="Never" />
     <disable_collisions link1="left_wrist" link2="left_hand" reason="Never" />
     <disable_collisions link1="left_wrist" link2="left_upper_forearm" reason="Never" />
@@ -146,5 +127,4 @@
     <disable_collisions link1="left_hand_range" link2="left_upper_forearm_visual" reason="Never" />
     <disable_collisions link1="left_hand_range" link2="left_wrist" reason="Never" />
-    <disable_collisions link1="left_hand_range" link2="right_gripper" reason="Never" />
     <disable_collisions link1="left_hand_range" link2="right_hand_camera" reason="Never" />
     <disable_collisions link1="left_hand_range" link2="right_hand_range" reason="Never" />
@@ -209,5 +189,4 @@
     <disable_collisions link1="left_upper_shoulder" link2="torso" reason="Adjacent" />
     <disable_collisions link1="pedestal" link2="right_hand_accelerometer" reason="Never" />
-    <disable_collisions link1="pedestal" link2="right_gripper_base" reason="Default" />
     <disable_collisions link1="pedestal" link2="right_hand_camera" reason="Default" />
     <disable_collisions link1="pedestal" link2="right_hand_range" reason="Default" />
@@ -219,5 +198,4 @@
     <disable_collisions link1="pedestal" link2="right_upper_shoulder" reason="Never" />
     <disable_collisions link1="pedestal" link2="left_hand_accelerometer" reason="Never" />
-    <disable_collisions link1="pedestal" link2="left_gripper_base" reason="Default" />
     <disable_collisions link1="pedestal" link2="left_hand_camera" reason="Default" />
     <disable_collisions link1="pedestal" link2="left_hand_range" reason="Default" />
@@ -231,20 +209,5 @@
     <disable_collisions link1="pedestal" link2="sonar_ring" reason="Never" />
     <disable_collisions link1="pedestal" link2="torso" reason="Adjacent" />
-    <disable_collisions link1="right_gripper" link2="right_hand" reason="Adjacent" />
-    <disable_collisions link1="right_gripper" link2="right_hand_camera" reason="Never" />
-    <disable_collisions link1="right_gripper" link2="right_hand_range" reason="Never" />
-    <disable_collisions link1="right_gripper" link2="right_lower_elbow" reason="Never" />
-    <disable_collisions link1="right_gripper" link2="right_lower_forearm" reason="Never" />
-    <disable_collisions link1="right_gripper" link2="right_upper_elbow" reason="Never" />
-    <disable_collisions link1="right_gripper" link2="right_upper_elbow_visual" reason="Never" />
-    <disable_collisions link1="right_gripper" link2="right_upper_forearm" reason="Never" />
-    <disable_collisions link1="right_gripper" link2="right_upper_forearm_visual" reason="Never" />
-    <disable_collisions link1="right_gripper" link2="right_wrist" reason="Never" />
-    <disable_collisions link1="right_gripper" link2="screen" reason="Never" />
-    <disable_collisions link1="right_gripper" link2="sonar_ring" reason="Never" />
-    <disable_collisions link1="right_gripper" link2="pedestal" reason="Never" />
-    <disable_collisions link1="right_gripper_base" link2="right_hand_accelerometer" reason="Never" />
     <disable_collisions link1="right_hand" link2="right_hand_accelerometer" reason="Never" />
-    <disable_collisions link1="right_hand" link2="right_gripper_base" reason="Adjacent" />
     <disable_collisions link1="right_hand" link2="right_hand_camera" reason="Adjacent" />
     <disable_collisions link1="right_hand" link2="right_hand_range" reason="Adjacent" />
@@ -272,5 +235,4 @@
     <disable_collisions link1="right_hand_range" link2="right_upper_forearm" reason="Never" />
     <disable_collisions link1="right_wrist" link2="right_hand_accelerometer" reason="Never" />
-    <disable_collisions link1="right_wrist" link2="right_gripper_base" reason="Never" />
     <disable_collisions link1="right_wrist" link2="right_upper_forearm" reason="Never" />
     <disable_collisions link1="right_wrist" link2="right_upper_forearm_visual" reason="Never" />

File: baxter/baxter_moveit_config/config/rethink_electric_gripper.srdf.xacro (robot description, xacro)
@@ -6,75 +6,59 @@
 <robot xmlns:xacro="http://www.ros.org/wiki/xacro" name="rethink_electric_gripper">
     <xacro:macro name="rethink_electric_gripper" params="side">
-    <disable_collisions link1="${side}_gripper_base" link2="${side}_gripper_electric_base" reason="Adjacent" />
-    <disable_collisions link1="${side}_gripper_base" link2="${side}_gripper_l_finger" reason="Never" />
-    <disable_collisions link1="${side}_gripper_base" link2="${side}_gripper_l_finger_tip" reason="Never" />
-    <disable_collisions link1="${side}_gripper_base" link2="${side}_gripper_r_finger" reason="Never" />
-    <disable_collisions link1="${side}_gripper_base" link2="${side}_gripper_r_finger_tip" reason="Never" />
-    <disable_collisions link1="${side}_gripper_electric_base" link2="${side}_gripper_l_finger" reason="Adjacent" />
-    <disable_collisions link1="${side}_gripper_electric_base" link2="${side}_gripper_l_finger_tip" reason="Never" />
-    <disable_collisions link1="${side}_gripper_electric_base" link2="${side}_gripper_r_finger" reason="Adjacent" />
-    <disable_collisions link1="${side}_gripper_electric_base" link2="${side}_gripper_r_finger_tip" reason="Never" />
-    <disable_collisions link1="${side}_gripper_electric_base" link2="${side}_hand" reason="Default" />
-    <disable_collisions link1="${side}_gripper_electric_base" link2="${side}_hand_accelerometer" reason="Never" />
-    <disable_collisions link1="${side}_gripper_electric_base" link2="${side}_hand_camera" reason="Default" />
-    <disable_collisions link1="${side}_gripper_electric_base" link2="${side}_hand_range" reason="Default" />
-    <disable_collisions link1="${side}_gripper_electric_base" link2="${side}_lower_elbow" reason="Never" />
-    <disable_collisions link1="${side}_gripper_electric_base" link2="${side}_lower_forearm" reason="Never" />
-    <disable_collisions link1="${side}_gripper_electric_base" link2="${side}_upper_elbow_visual" reason="Never" />
-    <disable_collisions link1="${side}_gripper_electric_base" link2="${side}_upper_forearm" reason="Never" />
-    <disable_collisions link1="${side}_gripper_electric_base" link2="${side}_upper_forearm_visual" reason="Never" />
-    <disable_collisions link1="${side}_gripper_electric_base" link2="${side}_wrist" reason="Never" />
-    <disable_collisions link1="${side}_gripper" link2="${side}_gripper_electric_base" reason="Default" />
-    <disable_collisions link1="${side}_gripper" link2="${side}_gripper_l_finger" reason="Default" />
-    <disable_collisions link1="${side}_gripper" link2="${side}_gripper_l_finger_tip" reason="Never" />
-    <disable_collisions link1="${side}_gripper" link2="${side}_gripper_r_finger" reason="Default" />
-    <disable_collisions link1="${side}_gripper" link2="${side}_gripper_r_finger_tip" reason="Never" />
-    <disable_collisions link1="${side}_gripper_l_finger" link2="${side}_gripper_l_finger_tip" reason="Adjacent" />
-    <disable_collisions link1="${side}_gripper_l_finger" link2="${side}_gripper_r_finger" reason="Never" />
-    <disable_collisions link1="${side}_gripper_l_finger" link2="${side}_gripper_r_finger_tip" reason="Never" />
-    <disable_collisions link1="${side}_gripper_l_finger" link2="${side}_hand" reason="Never" />
-    <disable_collisions link1="${side}_gripper_l_finger" link2="${side}_hand_accelerometer" reason="Never" />
-    <disable_collisions link1="${side}_gripper_l_finger" link2="${side}_hand_camera" reason="Never" />
-    <disable_collisions link1="${side}_gripper_l_finger" link2="${side}_hand_range" reason="Never" />
-    <disable_collisions link1="${side}_gripper_l_finger" link2="${side}_lower_elbow" reason="Never" />
-    <disable_collisions link1="${side}_gripper_l_finger" link2="${side}_lower_forearm" reason="Never" />
-    <disable_collisions link1="${side}_gripper_l_finger" link2="${side}_upper_forearm" reason="Never" />
-    <disable_collisions link1="${side}_gripper_l_finger" link2="${side}_upper_forearm_visual" reason="Never" />
-    <disable_collisions link1="${side}_gripper_l_finger" link2="${side}_wrist" reason="Never" />
-    <disable_collisions link1="${side}_gripper_l_finger_tip" link2="${side}_gripper_r_finger" reason="Never" />
-    <disable_collisions link1="${side}_gripper_l_finger_tip" link2="${side}_hand" reason="Never" />
-    <disable_collisions link1="${side}_gripper_l_finger_tip" link2="${side}_hand_accelerometer" reason="Never" />
-    <disable_collisions link1="${side}_gripper_l_finger_tip" link2="${side}_hand_camera" reason="Never" />
-    <disable_collisions link1="${side}_gripper_l_finger_tip" link2="${side}_hand_range" reason="Never" />
-    <disable_collisions link1="${side}_gripper_l_finger_tip" link2="${side}_lower_elbow" reason="Never" />
-    <disable_collisions link1="${side}_gripper_l_finger_tip" link2="${side}_lower_forearm" reason="Never" />
-    <disable_collisions link1="${side}_gripper_l_finger_tip" link2="${side}_upper_elbow_visual" reason="Never" />
-    <disable_collisions link1="${side}_gripper_l_finger_tip" link2="${side}_upper_forearm" reason="Never" />
-    <disable_collisions link1="${side}_gripper_l_finger_tip" link2="${side}_upper_forearm_visual" reason="Never" />
-    <disable_collisions link1="${side}_gripper_l_finger_tip" link2="${side}_wrist" reason="Never" />
-    <disable_collisions link1="${side}_gripper_r_finger" link2="${side}_gripper_r_finger_tip" reason="Adjacent" />
-    <disable_collisions link1="${side}_gripper_r_finger" link2="${side}_hand" reason="Never" />
-    <disable_collisions link1="${side}_gripper_r_finger" link2="${side}_hand_accelerometer" reason="Never" />
-    <disable_collisions link1="${side}_gripper_r_finger" link2="${side}_hand_camera" reason="Never" />
-    <disable_collisions link1="${side}_gripper_r_finger" link2="${side}_hand_range" reason="Never" />
-    <disable_collisions link1="${side}_gripper_r_finger" link2="${side}_lower_elbow" reason="Never" />
-    <disable_collisions link1="${side}_gripper_r_finger" link2="${side}_lower_forearm" reason="Never" />
-    <disable_collisions link1="${side}_gripper_r_finger" link2="${side}_upper_forearm" reason="Never" />
-    <disable_collisions link1="${side}_gripper_r_finger" link2="${side}_upper_forearm_visual" reason="Never" />
-    <disable_collisions link1="${side}_gripper_r_finger" link2="${side}_wrist" reason="Never" />
-    <disable_collisions link1="${side}_gripper_r_finger_tip" link2="${side}_hand" reason="Never" />
-    <disable_collisions link1="${side}_gripper_r_finger_tip" link2="${side}_hand_accelerometer" reason="Never" />
-    <disable_collisions link1="${side}_gripper_r_finger_tip" link2="${side}_hand_camera" reason="Never" />
-    <disable_collisions link1="${side}_gripper_r_finger_tip" link2="${side}_hand_range" reason="Never" />
-    <disable_collisions link1="${side}_gripper_r_finger_tip" link2="${side}_lower_elbow" reason="Never" />
-    <disable_collisions link1="${side}_gripper_r_finger_tip" link2="${side}_lower_forearm" reason="Never" />
-    <disable_collisions link1="${side}_gripper_r_finger_tip" link2="${side}_upper_elbow_visual" reason="Never" />
-    <disable_collisions link1="${side}_gripper_r_finger_tip" link2="${side}_upper_forearm" reason="Never" />
-    <disable_collisions link1="${side}_gripper_r_finger_tip" link2="${side}_upper_forearm_visual" reason="Never" />
-    <disable_collisions link1="${side}_gripper_r_finger_tip" link2="${side}_wrist" reason="Never" />
-    <disable_collisions link1="${side}_gripper_l_finger_tip" link2="${side}_gripper_r_finger_tip" reason="Never" />
-    <disable_collisions link1="${side}_gripper_l_finger" link2="${side}_gripper_l_finger_tip" reason="Never" />
-    <disable_collisions link1="${side}_gripper_r_finger" link2="${side}_gripper_r_finger_tip" reason="Never" />
-    <disable_collisions link1="${side}_gripper_base" link2="${side}_gripper_electric_base" reason="Never" />
+    <xacro:property name="gripper_side" value="${side[0]}" scope="local"/>
+    <disable_collisions link1="${side}_gripper_base" link2="${gripper_side}_gripper_l_finger" reason="Adjacent" />
+    <disable_collisions link1="${side}_gripper_base" link2="${gripper_side}_gripper_l_finger_tip" reason="Never" />
+    <disable_collisions link1="${side}_gripper_base" link2="${gripper_side}_gripper_r_finger" reason="Adjacent" />
+    <disable_collisions link1="${side}_gripper_base" link2="${gripper_side}_gripper_r_finger_tip" reason="Never" />
+    <disable_collisions link1="${side}_gripper" link2="${gripper_side}_gripper_l_finger" reason="Default" />
+    <disable_collisions link1="${side}_gripper" link2="${gripper_side}_gripper_l_finger_tip" reason="Never" />
+    <disable_collisions link1="${side}_gripper" link2="${gripper_side}_gripper_r_finger" reason="Default" />
+    <disable_collisions link1="${side}_gripper" link2="${gripper_side}_gripper_r_finger_tip" reason="Never" />
+    <disable_collisions link1="${gripper_side}_gripper_l_finger" link2="${gripper_side}_gripper_l_finger_tip" reason="Adjacent" />
+    <disable_collisions link1="${gripper_side}_gripper_l_finger" link2="${gripper_side}_gripper_r_finger" reason="Never" />
+    <disable_collisions link1="${gripper_side}_gripper_l_finger" link2="${gripper_side}_gripper_r_finger_tip" reason="Never" />
+    <disable_collisions link1="${gripper_side}_gripper_l_finger" link2="${side}_hand" reason="Never" />
+    <disable_collisions link1="${gripper_side}_gripper_l_finger" link2="${side}_hand_accelerometer" reason="Never" />
+    <disable_collisions link1="${gripper_side}_gripper_l_finger" link2="${side}_hand_camera" reason="Never" />
+    <disable_collisions link1="${gripper_side}_gripper_l_finger" link2="${side}_hand_range" reason="Never" />
+    <disable_collisions link1="${gripper_side}_gripper_l_finger" link2="${side}_lower_elbow" reason="Never" />
+    <disable_collisions link1="${gripper_side}_gripper_l_finger" link2="${side}_lower_forearm" reason="Never" />
+    <disable_collisions link1="${gripper_side}_gripper_l_finger" link2="${side}_upper_forearm" reason="Never" />
+    <disable_collisions link1="${gripper_side}_gripper_l_finger" link2="${side}_upper_forearm_visual" reason="Never" />
+    <disable_collisions link1="${gripper_side}_gripper_l_finger" link2="${side}_wrist" reason="Never" />
+    <disable_collisions link1="${gripper_side}_gripper_l_finger_tip" link2="${gripper_side}_gripper_r_finger" reason="Never" />
+    <disable_collisions link1="${gripper_side}_gripper_l_finger_tip" link2="${side}_hand" reason="Never" />
+    <disable_collisions link1="${gripper_side}_gripper_l_finger_tip" link2="${side}_hand_accelerometer" reason="Never" />
+    <disable_collisions link1="${gripper_side}_gripper_l_finger_tip" link2="${side}_hand_camera" reason="Never" />
+    <disable_collisions link1="${gripper_side}_gripper_l_finger_tip" link2="${side}_hand_range" reason="Never" />
+    <disable_collisions link1="${gripper_side}_gripper_l_finger_tip" link2="${side}_lower_elbow" reason="Never" />
+    <disable_collisions link1="${gripper_side}_gripper_l_finger_tip" link2="${side}_lower_forearm" reason="Never" />
+    <disable_collisions link1="${gripper_side}_gripper_l_finger_tip" link2="${side}_upper_elbow_visual" reason="Never" />
+    <disable_collisions link1="${gripper_side}_gripper_l_finger_tip" link2="${side}_upper_forearm" reason="Never" />
+    <disable_collisions link1="${gripper_side}_gripper_l_finger_tip" link2="${side}_upper_forearm_visual" reason="Never" />
+    <disable_collisions link1="${gripper_side}_gripper_l_finger_tip" link2="${side}_wrist" reason="Never" />
+    <disable_collisions link1="${gripper_side}_gripper_r_finger" link2="${gripper_side}_gripper_r_finger_tip" reason="Adjacent" />
+    <disable_collisions link1="${gripper_side}_gripper_r_finger" link2="${side}_hand" reason="Never" />
+    <disable_collisions link1="${gripper_side}_gripper_r_finger" link2="${side}_hand_accelerometer" reason="Never" />
+    <disable_collisions link1="${gripper_side}_gripper_r_finger" link2="${side}_hand_camera" reason="Never" />
+    <disable_collisions link1="${gripper_side}_gripper_r_finger" link2="${side}_hand_range" reason="Never" />
+    <disable_collisions link1="${gripper_side}_gripper_r_finger" link2="${side}_lower_elbow" reason="Never" />
+    <disable_collisions link1="${gripper_side}_gripper_r_finger" link2="${side}_lower_forearm" reason="Never" />
+    <disable_collisions link1="${gripper_side}_gripper_r_finger" link2="${side}_upper_forearm" reason="Never" />
+    <disable_collisions link1="${gripper_side}_gripper_r_finger" link2="${side}_upper_forearm_visual" reason="Never" />
+    <disable_collisions link1="${gripper_side}_gripper_r_finger" link2="${side}_wrist" reason="Never" />
+    <disable_collisions link1="${gripper_side}_gripper_r_finger_tip" link2="${side}_hand" reason="Never" />
+    <disable_collisions link1="${gripper_side}_gripper_r_finger_tip" link2="${side}_hand_accelerometer" reason="Never" />
+    <disable_collisions link1="${gripper_side}_gripper_r_finger_tip" link2="${side}_hand_camera" reason="Never" />
+    <disable_collisions link1="${gripper_side}_gripper_r_finger_tip" link2="${side}_hand_range" reason="Never" />
+    <disable_collisions link1="${gripper_side}_gripper_r_finger_tip" link2="${side}_lower_elbow" reason="Never" />
+    <disable_collisions link1="${gripper_side}_gripper_r_finger_tip" link2="${side}_lower_forearm" reason="Never" />
+    <disable_collisions link1="${gripper_side}_gripper_r_finger_tip" link2="${side}_upper_elbow_visual" reason="Never" />
+    <disable_collisions link1="${gripper_side}_gripper_r_finger_tip" link2="${side}_upper_forearm" reason="Never" />
+    <disable_collisions link1="${gripper_side}_gripper_r_finger_tip" link2="${side}_upper_forearm_visual" reason="Never" />
+    <disable_collisions link1="${gripper_side}_gripper_r_finger_tip" link2="${side}_wrist" reason="Never" />
+    <disable_collisions link1="${gripper_side}_gripper_l_finger_tip" link2="${gripper_side}_gripper_r_finger_tip" reason="Never" />
+    <disable_collisions link1="${gripper_side}_gripper_l_finger" link2="${gripper_side}_gripper_l_finger_tip" reason="Never" />
+    <disable_collisions link1="${gripper_side}_gripper_r_finger" link2="${gripper_side}_gripper_r_finger_tip" reason="Never" />
     </xacro:macro>
 </robot>
